File: uv_matrix.kicad_pcb (KiCad board)
At the start: 2 copper layers, 255.3 x 190.5 mm, 240 parts

Commit message: dgdgd
Parts:
- removed D100, D101, D102, D103, D104, D105, D106, D107, D108, D109, D110, D111, D112, D113, D114, D115, D116, D117, D118, D119, D120, D121, D122, D123, D124, D125, D126, D127, D128, D129, D130, D131, D132, D133, D134, D135, D136, D137, D138, D139, D140, D141, D142, D143, D144, D145, D146, D147, D148, D149, D150, D151, D152, D153, D154, D155, D156, D157, D158, D159, D160, D161, D162, D163, D164, D165, D166, D167, D168, D169, D170, D171, D172, D173, D174, D175, D176, D177, D178, D179, D180, D65, D66, D67, D68, D69, D70, D71, D72, D73, D74, D75, D76, D77, D78, D79, D80, D81, D82, D83, D84, D85, D86, D87, D88, D89, D90, D91, D92, D93, D94, D95, D96, D97, D98, D99: LED, LEDs:LED-5MM
- removed R1, R10, R11, R12, R13, R14, R15, R16, R17, R18, R19, R2, R20, R21, R22, R23, R24, R25, R26, R27, R28, R29, R3, R30, R31, R32, R33, R34, R35, R36, R37, R38, R39, R4, R40, R41, R42, R43, R44, R45, R46, R47, R48, R49, R5, R50, R51, R52, R53, R54, R55, R56, R57, R58, R59, R6, R60, R7, R8, R9: 100, Resistors_ThroughHole:Resistor_Horizontal_RM10mm
- moved D9 278.3 mm to (17.8, 40.6), turned to 0 degrees
- moved D10 272.8 mm to (35.6, 40.6), turned to 0 degrees
- moved D11 269.1 mm to (53.3, 40.6), turned to 0 degrees
- moved D12 267.4 mm to (71.1, 40.6), turned to 0 degrees
- moved D1 237.4 mm to (17.8, 22.9), turned to 0 degrees
- moved D17 229.7 mm to (17.8, 58.4), turned to 0 degrees
- moved D33 225.5 mm to (17.8, 94.0), turned to 0 degrees
- moved D2 224.1 mm to (35.6, 22.9), turned to 0 degrees
- moved D18 218.9 mm to (35.6, 58.4), turned to 0 degrees
- moved D34 217.4 mm to (35.6, 94.0), turned to 0 degrees
- moved D3 212.6 mm to (53.3, 22.9), turned to 0 degrees
- moved D35 211.5 mm to (53.3, 94.0), turned to 0 degrees
- moved D19 210.1 mm to (53.3, 58.4), turned to 0 degrees
- moved D36 208.1 mm to (71.1, 94.0), turned to 0 degrees
- moved D24 203.6 mm to (142.2, 58.4), turned to 0 degrees
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Connections:
- D1 pad 1: Net-(D1-Pad1) -> GNDREF
- D12 pad 2: GNDREF -> +12V
- D13 pad 1: Net-(D13-Pad1) -> GNDREF
- D15 pad 2: GNDREF -> Net-(D15-Pad2)
- D16 pad 1: Net-(D16-Pad1) -> Net-(D15-Pad2)
- D16 pad 2: Net-(D16-Pad2) -> +12V
- D17 pad 1: Net-(D16-Pad2) -> GNDREF
- D18 pad 2: GNDREF -> Net-(D18-Pad2)
- D19 pad 1: Net-(D19-Pad1) -> Net-(D18-Pad2)
- D20 pad 2: Net-(D20-Pad2) -> +12V
- D21 pad 1: Net-(D20-Pad2) -> GNDREF
- D21 pad 2: GNDREF -> Net-(D21-Pad2)
- D22 pad 1: Net-(D22-Pad1) -> Net-(D21-Pad2)
- D24 pad 2: GNDREF -> +12V
- D25 pad 1: Net-(D25-Pad1) -> GNDREF
- D27 pad 2: GNDREF -> Net-(D27-Pad2)
- D28 pad 1: Net-(D28-Pad1) -> Net-(D27-Pad2)
- D28 pad 2: Net-(D28-Pad2) -> +12V
- D29 pad 1: Net-(D28-Pad2) -> GNDREF
- D3 pad 2: GNDREF -> Net-(D3-Pad2)
- D30 pad 2: GNDREF -> Net-(D30-Pad2)
- D31 pad 1: Net-(D31-Pad1) -> Net-(D30-Pad2)
- D32 pad 2: Net-(D32-Pad2) -> +12V
- D33 pad 1: Net-(D32-Pad2) -> GNDREF
- D33 pad 2: GNDREF -> Net-(D33-Pad2)
- D34 pad 1: Net-(D34-Pad1) -> Net-(D33-Pad2)
- D36 pad 2: GNDREF -> +12V
- D37 pad 1: Net-(D37-Pad1) -> GNDREF
- D39 pad 2: GNDREF -> Net-(D39-Pad2)
- D4 pad 1: Net-(D4-Pad1) -> Net-(D3-Pad2)
- D4 pad 2: Net-(D4-Pad2) -> +12V
- D40 pad 1: Net-(D40-Pad1) -> Net-(D39-Pad2)
- D40 pad 2: Net-(D40-Pad2) -> +12V
- D41 pad 1: Net-(D40-Pad2) -> GNDREF
- D42 pad 2: GNDREF -> Net-(D42-Pad2)
- D43 pad 1: Net-(D43-Pad1) -> Net-(D42-Pad2)
- D44 pad 2: Net-(D44-Pad2) -> +12V
- D45 pad 1: Net-(D44-Pad2) -> GNDREF
- D45 pad 2: GNDREF -> Net-(D45-Pad2)
- D46 pad 1: Net-(D46-Pad1) -> Net-(D45-Pad2)
- D48 pad 2: GNDREF -> +12V
- D49 pad 1: Net-(D49-Pad1) -> GNDREF
- D5 pad 1: Net-(D4-Pad2) -> GNDREF
- D51 pad 2: GNDREF -> Net-(D51-Pad2)
- D52 pad 1: Net-(D52-Pad1) -> Net-(D51-Pad2)
- D52 pad 2: Net-(D52-Pad2) -> +12V
- D53 pad 1: Net-(D52-Pad2) -> GNDREF
- D54 pad 2: GNDREF -> Net-(D54-Pad2)
- D55 pad 1: Net-(D55-Pad1) -> Net-(D54-Pad2)
- D56 pad 2: Net-(D56-Pad2) -> +12V
- D57 pad 1: Net-(D56-Pad2) -> GNDREF
- D57 pad 2: GNDREF -> Net-(D57-Pad2)
- D58 pad 1: Net-(D58-Pad1) -> Net-(D57-Pad2)
- D6 pad 2: GNDREF -> Net-(D6-Pad2)
- D60 pad 2: GNDREF -> +12V
- D61 pad 1: Net-(D61-Pad1) -> GNDREF
- D63 pad 2: GNDREF -> Net-(D63-Pad2)
- D64 pad 1: Net-(D64-Pad1) -> Net-(D63-Pad2)
- D64 pad 2: Net-(D64-Pad2) -> +12V
- D7 pad 1: Net-(D7-Pad1) -> Net-(D6-Pad2)
- D8 pad 2: Net-(D8-Pad2) -> +12V
- D9 pad 1: Net-(D8-Pad2) -> GNDREF
- D9 pad 2: GNDREF -> Net-(D10-Pad1)
Routing:
- net GNDREF: track 0.00 -> 384.1 mm
- net +12V: track 0.00 -> 351.1 mm
- net Net-(D7-Pad2): track 0.00 -> 15.2 mm
- net Net-(D63-Pad2): track 0.00 -> 15.2 mm
- net Net-(D61-Pad2): track 0.00 -> 15.2 mm
- net Net-(D55-Pad2): track 0.00 -> 15.2 mm
- net Net-(D53-Pad2): track 0.00 -> 15.2 mm
- net Net-(D5-Pad2): track 0.00 -> 15.2 mm
- net Net-(D47-Pad2): track 0.00 -> 15.2 mm
- net Net-(D45-Pad2): track 0.00 -> 15.2 mm
- net Net-(D39-Pad2): track 0.00 -> 15.2 mm
- net Net-(D37-Pad2): track 0.00 -> 15.2 mm
- net Net-(D31-Pad2): track 0.00 -> 15.2 mm
- net Net-(D29-Pad2): track 0.00 -> 15.2 mm
- net Net-(D23-Pad2): track 0.00 -> 15.2 mm
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Other:
- board size 255.3 x 190.5 mm -> 139.7 x 149.9 mm
- net class Default: trace_width 0.25 -> 0.6
